File: Analog Shield/Kicad/AnalogFrontEnd/AnalogFrontEnd.kicad_sch (KiCad schematic)
At the start: 23 parts

Commit message: Analog front end schematic finished draft
Parts:
- removed R?: 90.9KΩ, symbol Device:R
- removed R? (x2): 100Ω, symbol Device:R
- removed R? (x2): 1MΩ, symbol Device:R
- removed R?: 402Ω, symbol Device:R
- removed R? (x2): 10KΩ, symbol Device:R
- removed R? (x2): 10MΩ, symbol Device:R
- removed R?: 604Ω, symbol Device:R
- removed U? (x2): ADG1236YRUZ, RU_16_ADI, symbol New_Library:ADG1236YRUZ
- removed U? (x2): AD8420ARMZ-R7, SOP65P490X110-8N, symbol New_Library:AD8420ARMZ-R7
- removed U?: AD823ARZ-RL, R_8_ADI, symbol New_Library:AD823ARZ-RL
- removed U? (x2): ADG509FBRUZ, RU_16_ADI, symbol New_Library:ADG509FBRUZ
- added J?: Interface, symbol Connector_Generic:Conn_01x06
Connections:
- net +5V: now also J?.5 (Pin_5)
- net GND: now also J?.6 (Pin_6)
- new net DUT1+: J?.1 (Pin_1)
- new net DUT1-: J?.2 (Pin_2)
- new net DUT2+: J?.3 (Pin_3)
- new net DUT2-: J?.4 (Pin_4)
- no-connect marks 12 -> 2
Other:
- added sheet Channel 1 (Channel1.kicad_sch)
- added sheet Channel 2 (Channel2.kicad_sch)
- moved on the sheet: J?

Commit message: Analog Shield Layout Draft
Parts:
- added C1, C2, C3, C4, C5, C6, C7, C8: 10μF, Library:0603, symbol Device:C
- added JP1, JP2: SolderJumper_2_Open, Jumper:SolderJumper-2_P1.3mm_Open_RoundedPad1.0x1.5mm, symbol Jumper:SolderJumper_2_Open
- added R1, R2, R3, R4, R5, R6, R7, R8: 10KΩ, Library:0603, symbol Device:R
- added U1, U2, U3, U4: AD8130ARMZ-REEL7, Library:AD8130, symbol New_Library:AD8130ARMZ-REEL7
- J1, J2, J3, J4: renamed from J?; footprint (none) -> Connector_PinHeader_2.54mm:PinHeader_1x08_P2.54mm_Vertical
- J5, J6: renamed from J?; footprint (none) -> Connector_PinHeader_2.54mm:PinHeader_1x06_P2.54mm_Vertical
Connections:
- net +12V: now also C3.2, C4.2, C7.2, C8.2, U1.3 (PD*), U1.7 (+VS), U2.3 (PD*), U2.7 (+VS), U3.3 (PD*), U3.7 (+VS), U4.3 (PD*), U4.7 (+VS)
- net -12V: now also C1.2, C2.2, C5.2, C6.2, U1.2 (-VS), U2.2 (-VS), U3.2 (-VS), U4.2 (-VS)
- net CH1IN+: now also R1.2, R3.1
- net CH1IN-: now also R2.2, R4.1
- net CH2IN+: now also R5.2, R7.1
- net CH2IN-: now also R6.2, R8.1
- net GND: now also C1.1, C2.1, C3.1, C4.1, C5.1, C6.1, C7.1, C8.1, R1.1, R2.1, R5.1, R6.1
- net VREF: now also JP1.2 (B), JP2.2 (B), U1.5 (FB), U2.5 (FB), U3.5 (FB), U4.5 (FB)
- new net: JP2.1 (A), R8.2, U4.4 (REF), U4.6 (OUT)
- new net: R3.2, U1.4 (REF), U1.6 (OUT)
- new net: JP1.1 (A), R4.2, U2.4 (REF), U2.6 (OUT)
- new net: R7.2, U3.4 (REF), U3.6 (OUT)
- new net CH1_VDM+: U1.1 (+IN), U2.8 (-IN)
- new net CH1_VDM-: U1.8 (-IN), U2.1 (+IN)
- new net CH2_VDM+: U3.1 (+IN), U4.8 (-IN)
- new net CH2_VDM-: U3.8 (-IN), U4.1 (+IN)
Other:
- sheet Channel 1 ports: added CH1_EN, CH1_I0, CH1_I1, CH1_MV, CH1_SI, CH2_I0, CH2_I1; removed D0, D1, D2, D3, D4, D8, D9
- sheet Channel 2 ports: added CH2_ENA, CH2_I0, CH2_I1, CH2_MV, CH2_SI; removed D10, D11, D7, D8, D9
- moved on the sheet: J1, J2, J3, J4, J5, J6
