File: Analog Shield/Kicad/AnalogFrontEnd/Channel1.kicad_sch (KiCad schematic)
At the start: 55 parts

Commit message: Analog Shield Layout Draft
Parts:
- removed C? (x4): 1μF, symbol Device:C
- removed C? (x4): 0.1μF, symbol Device:C
- C10, C11, C12, C13, C14, C15, C16, C17, C18, C19, C20, C21, C22, C23, C24, C25, C26, C27, C28, C29, C30, C31, C32, C9: renamed from C?; footprint (none) -> Library:0603
- R10, R11, R12, R13, R14, R16, R17, R18, R9: renamed from R?; footprint (none) -> Library:0603
- R15, R19: renamed from R?; footprint (none) -> Library:1206
- U10: renamed from U?; footprint DCK5 -> Library:SN74AHCT1G32
- U11, U12: renamed from U?; footprint RU_16_ADI -> Library:ADG509F
- U13: renamed from U?; footprint RM_8_ADI -> Library:AD823
- U14: renamed from U?; footprint DB16 -> Library:SN74HC139
- U15: renamed from U?; footprint RU_16_ADI -> Library:ADG411
- U16: renamed from U?; footprint DBV0005A_N -> Library:SN74LVC1G08
- U5, U8: renamed from U?; footprint RM_8_ADI -> Library:AD8130
- U6, U7: renamed from U?; footprint RU_16_ADI -> Library:ADG1236
- U9: renamed from U?; footprint DCK0005A_N -> Library:SN74AHCT1G04
Connections:
- net D9 is gone; now on net CH2Y: U14.15 (*2G)
- net S22 is gone; now on net S2B: U14.11 (2Y1)
- net S23 is gone; now on net S2A: U14.12 (2Y0)
- net CH2Y: no longer U14.13 (2B)
- net S2A: no longer U14.10 (2Y2)
- net S2B: no longer U14.9 (2Y3)
- net at U10.4 (Y): now also U14.1 (*1G); no longer U14.3 (1B)
- net at U16.1 (A): now also U14.4 (1Y0); no longer U14.6 (1Y2)
- net at U16.2 (B): now also U14.5 (1Y1); no longer U14.7 (1Y3)
- net +5V renamed +3V3
- net D0 renamed CH1_EN
- net D1 renamed CH1_I1
- net CH1_I1: now also U14.3 (1B); no longer U14.2 (1A)
- net D2 renamed CH1_I0
- net CH1_I0: now also U14.2 (1A); no longer U14.1 (*1G)
- net D3 renamed CH1_SI
- net D4 renamed CH1_MV
- net D8 renamed CH2_I0
- net S11 renamed S1_01
- net S12 renamed S1_2
- net S1_2: now also U14.6 (1Y2); no longer U14.5 (1Y1)
- net S13 renamed S1_3
- net S1_3: now also U14.7 (1Y3); no longer U14.4 (1Y0)
- new net CH2_I1: U14.13 (2B)
- new net S2_2: U14.10 (2Y2)
- new net S2_3: U14.9 (2Y3)
Other:
- moved on the sheet: C13, C14, C16, C17, C31, U16
