File: Analog Shield/Kicad/AnalogFrontEnd/Channel2.kicad_sch (KiCad schematic)
At the start: 52 parts

Commit message: Analog Shield Layout Draft
Parts:
- removed C? (x30): (no value), symbol Device:C
- removed R? (x11): (no value), symbol Device:R
- removed U? (x2): (no value), symbol New_Library:ADG1236YRUZ
- removed U? (x2): (no value), symbol New_Library:ADG509FBRUZ
- removed U?: (no value), symbol New_Library:AD823AARMZ
- removed U? (x2): (no value), symbol New_Library:AD8130ARMZ-REEL7
- removed U?: (no value), symbol New_Library:SN74AHCT1G04DCKR
- removed U?: (no value), symbol New_Library:SN74LVC1G08DBVR
- removed U?: (no value), symbol New_Library:SN74AHCT1G32DCKR
- removed U?: (no value), symbol New_Library:ADG411BRUZ
- added C33, C34, C35, C36, C39, C42, C43, C44, C45, C46, C47, C48, C52, C53, C54, C55: 0.1μF, Library:0603, symbol Device:C
- added C37, C38, C40, C41: 10μF, Library:0603, symbol Device:C
- added C49: 1μF, Library:0603, symbol Device:C
- added C50: 100nF, Library:0603, symbol Device:C
- added C51: 10nF, Library:0603, symbol Device:C
- added R20: 402Ω, Library:0603, symbol Device:R
- added R21, R23, R27: 100Ω, Library:0603, symbol Device:R
- added R22: 80.8KΩ, Library:0603, symbol Device:R
- added R24, R28: 10KΩ, Library:0603, symbol Device:R
- added R25, R29: 1MΩ, Library:0603, symbol Device:R
- added R26, R30: 10MΩ, Library:1206, symbol Device:R
- added U17, U20: AD8130ARMZ-REEL7, Library:AD8130, symbol New_Library:AD8130ARMZ-REEL7
- added U18, U19: ADG1236YRUZ, Library:ADG1236, symbol New_Library:ADG1236YRUZ
- added U21: SN74AHCT1G04DCKR, Library:SN74AHCT1G04, symbol New_Library:SN74AHCT1G04DCKR
- added U22: SN74AHCT1G32DCKR, Library:SN74AHCT1G32, symbol New_Library:SN74AHCT1G32DCKR
- added U23, U24: ADG509FBRUZ, Library:ADG509F, symbol New_Library:ADG509FBRUZ
- added U25: AD823AARMZ, Library:AD823, symbol New_Library:AD823AARMZ
- added U26: ADG411BRUZ, Library:ADG411, symbol New_Library:ADG411BRUZ
- added U27: SN74LVC1G08DBVR, Library:SN74LVC1G08, symbol New_Library:SN74LVC1G08DBVR
Connections:
- net +12V: now also C33.2, C34.2, C37.2, C40.2, C42.2, C43.2, C47.2, C52.2, U17.3 (PD*), U17.7 (+VS), U18.13 (VDD), U19.13 (VDD), U20.3 (PD*), U20.7 (+VS), U23.14 (VDD), U24.14 (VDD), U25.8 (VS+), U26.13 (VDD)
- net -12V: now also C35.2, C36.2, C38.2, C41.2, C44.2, C45.2, C48.2, C55.2, U17.2 (-VS), U18.5 (VSS), U19.5 (VSS), U20.2 (-VS), U23.3 (VSS), U24.3 (VSS), U25.4 (VS-), U26.4 (VSS)
- net CH2IN+: now also U19.3 (D1)
- net CH2IN-: now also U19.11 (D2)
- net CH2OUT+: now also U17.1 (+IN)
- net CH2OUT-: now also U17.8 (-IN)
- net CH2Y: now also U22.4 (Y)
- net DUT2+: now also C49.1, C50.1, C51.1, R27.2, R28.2, R29.2, R30.2, U25.3 (IN1+)
- net DUT2-: now also R23.2, R24.2, R25.2, R26.2, U25.5 (IN2+)
- net GND: now also C33.1, C34.1, C35.1, C36.1, C37.1, C38.1, C39.1, C40.1, C41.1, C42.1, C43.1, C44.1, C45.1, C46.1, C47.1, C48.1, C52.1, C53.1, C54.1, C55.1, U18.6 (GND), U19.6 (GND), U21.3 (GND), U22.3 (GND), U23.15 (GND), U24.15 (GND), U26.5 (GND), U27.3 (V-)
- net S2A: now also U27.1 (A)
- net S2B: now also U27.2 (B)
- new net: R29.1, U24.11 (S3B), U24.6 (S3A)
- new net: C50.2, U26.14 (S2)
- new net: R20.1, R21.2, R22.1, U18.10 (S2A), U19.2 (S1A)
- new net: U17.5 (FB), U18.11 (D2)
- new net: R21.1, U18.12 (S2B), U19.4 (S1B), U20.5 (FB), U25.6 (IN2-), U25.7 (OUT2), U26.10 (D3), U26.15 (D2), U26.2 (D1)
- new net: U18.2 (S1A), U19.10 (S2A), U20.8 (-IN), U24.9 (DB)
- new net: U17.4 (REF), U18.3 (D1)
- new net: R20.2, R22.2, U18.4 (S1B), U19.12 (S2B), U20.1 (+IN), U25.1 (OUT1), U25.2 (IN1-)
- new net: U20.4 (REF), U23.9 (DB)
- new net: U20.6 (OUT), U23.8 (DA)
- new net: C49.2, U26.3 (S1)
- new net: R30.1, U24.10 (S4B), U24.7 (S4A)
- new net: R26.1, U23.10 (S4B), U23.7 (S4A)
- new net: R28.1, U24.12 (S2B), U24.5 (S2A)
- new net: U21.4 (Y), U22.2 (B)
- new net: C51.2, U26.11 (S3)
- new net: R25.1, U23.11 (S3B), U23.6 (S3A)
- new net: R24.1, U23.12 (S2B), U23.5 (S2A)
- new net: R23.1, U23.13 (S1B), U23.4 (S1A)
- new net: R27.1, U24.13 (S1B), U24.4 (S1A)
- new net: U17.6 (OUT), U24.8 (DA)
- new net +3V3: C39.2, C46.2, C53.2, C54.2, U21.5 (VCC), U22.5 (VCC), U26.12 (VL), U27.5 (V+)
- new net CH2_ENA: U21.2 (A), U23.2 (EN), U24.2 (EN)
- new net CH2_I0: U23.1 (A0), U24.1 (A0)
- new net CH2_I1: U23.16 (A1), U24.16 (A1)
- new net CH2_MV: U19.1 (IN1), U19.9 (IN2)
- new net CH2_SI: U18.1 (IN1), U18.9 (IN2), U22.1 (A)
- new net S2_1: U26.1 (IN1), U27.4 (Y)
- new net S2_2: U26.16 (IN2)
- new net S2_3: U26.9 (IN3)
